File: schematic/kicad/circuit.sch (KiCad schematic (older format))
At the start: 20 parts, among them P1 Header 28, P2 Header 28, P3 Header 6, Q1 BC547

Commit message: doc: Update schemes
Signed-off-by: Mark Sungurov <mark.sungurov@gmail.com>
Parts:
- renumbered R4 to R1, R7 to R2, R6 to R3, R5 to R4, R3 to R5, R1 to R6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
Connections:
- net USART1_Tx renamed USART1_TX
Other:
- moved on the sheet: BTN1, BTN2, BTN3, BTN4, C1, P3, PiezoelectricBuzzer1, Q1, R2, R3, R4, R5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
